Commit message: urdf/path

File: install/sad_pkg/share/sad_pkg/urdf/description/test.xacro (robot description, xacro)
@@ -4,8 +4,33 @@
     <link name="world"/>
     <joint name="fixed_base" type="fixed" disable_fixed_joint_lumping="true">
-        <origin rpy="1.57 0 -1.57" xyz="0 -0.03 0"/>
+        <origin rpy="0 0 0" xyz="0 -0.03 0.0145"/>
         <parent link="world"/>
+        <child link="box_link"/>
+    </joint>
+    <joint name="fixed_base2" type="fixed" disable_fixed_joint_lumping="true">
+        <origin rpy="1.57 0 -1.57" xyz="0 0 0"/>
+        <parent link="box_link"/>
         <child link="base_link"/>
     </joint>
+    <!-- 박스 요소 추가 -->
+    <link name="box_link">
+        <visual>
+        <geometry>
+            <box size="0.25 0.25 0.029"/> <!-- x, y, z 크기 -->
+        </geometry>
+        <material name="grey"/>
+        </visual>
+        <collision>
+        <geometry>
+            <box size="0.25 0.25 0.029"/>
+        </geometry>
+        </collision>
+        <inertial>
+            <mass value="0.001"/>
+            <inertia ixx="0.01" ixy="0.0" ixz="0.0"
+                    iyy="0.01" iyz="0.0"
+                    izz="0.01"/>
+        </inertial>
+    </link>
     <link name="base_link">
         <visual>

Commit message: “deadbandX”

File: install/sad_pkg/share/sad_pkg/urdf/description/test.xacro (robot description, xacro)
@@ -4,10 +4,10 @@
     <link name="world"/>
     <joint name="fixed_base" type="fixed" disable_fixed_joint_lumping="true">
-        <origin rpy="0 0 0" xyz="0 -0.03 0.0145"/>
+        <origin rpy="0 0 0" xyz="0 -0.04 0.0145"/>
         <parent link="world"/>
         <child link="box_link"/>
     </joint>
     <joint name="fixed_base2" type="fixed" disable_fixed_joint_lumping="true">
-        <origin rpy="1.57 0 -1.57" xyz="0 0 0"/>
+        <origin rpy="1.57 0 -1.57" xyz="0 0 0.015"/>
         <parent link="box_link"/>
         <child link="base_link"/>
@@ -17,5 +17,5 @@
         <visual>
         <geometry>
-            <box size="0.25 0.25 0.029"/> <!-- x, y, z 크기 -->
+            <box size="0.25 0.25 0.029"/>
         </geometry>
         <material name="grey"/>
@@ -182,5 +182,5 @@
         <origin xyz="-0.044 0.383 -0.001" rpy="0 1.57 0"/>
         <axis xyz="0 1 0" />
-        <limit effort="1000.0" velocity="0.1" lower="-1.57" upper="1.57" />
+        <limit effort="1000.0" velocity="10" lower="-3.14" upper="3.14" />
         <dynamics damping="100" friction="50" />
     </joint>
@@ -189,6 +189,6 @@
         <child link="link2"/>
         <origin xyz="-0.004 0.018 0" rpy="0 0 0"/>
-        <axis xyz="0 0 1" />
-        <limit effort="1000.0" velocity="0.1" lower="-1.57" upper="1.57" />
+        <axis xyz="0 0 -1" />
+        <limit effort="1000.0" velocity="10" lower="-3.14" upper="3.14" />
         <dynamics damping="100" friction="50" />
     </joint>
@@ -198,5 +198,5 @@
         <origin xyz="0 0.205 0" rpy="0 3.14 3.14"/>
         <axis xyz="0 1 0" />
-        <limit effort="1000.0" velocity="0.1" lower="-1.57" upper="1.57" />
+        <limit effort="1000.0" velocity="10" lower="-3.14" upper="3.14" />
         <dynamics damping="100" friction="50" />
     </joint>
@@ -205,6 +205,6 @@
         <child link="link4"/>
         <origin xyz="0 -0.068 0.0015" rpy="-1.57 0 0"/>
-        <axis xyz="0 1 0" />
-        <limit effort="1000.0" velocity="0.1" lower="-1.57" upper="1.57" />
+        <axis xyz="0 -1 0" />
+        <limit effort="1000.0" velocity="10" lower="-3.14" upper="3.14" />
         <dynamics damping="100" friction="50" />
     </joint>
@@ -214,5 +214,5 @@
         <origin xyz="0 0.0005 -0.202" rpy="1.57 0 1.57"/>
         <axis xyz="0 1 0" />
-        <limit effort="1000.0" velocity="0.1" lower="-1.57" upper="1.57" />
+        <limit effort="1000.0" velocity="10" lower="-3.14" upper="3.14" />
         <dynamics damping="100" friction="50" />
     </joint>
@@ -221,6 +221,6 @@
         <child link="link6"/>
         <origin xyz="0 -0.053 0" rpy="1.57 1.57 0"/>
-        <axis xyz="0 1 0" />
-        <limit effort="1000.0" velocity="0.1" lower="-1.57" upper="1.57" />
+        <axis xyz="0 -1 0" />
+        <limit effort="1000.0" velocity="10" lower="-3.14" upper="3.14" />
         <dynamics damping="100" friction="50" />
     </joint>
@@ -230,5 +230,5 @@
         <origin xyz="-0.086 0.002 0.04" rpy="-1.57 0 3.14"/>
         <axis xyz="0 1 0" />
-        <limit effort="1000.0" velocity="0.1" lower="-1.57" upper="1.57" />
+        <limit effort="1000.0" velocity="10" lower="-3.14" upper="3.14" />
         <dynamics damping="100" friction="50" />
     </joint>

Commit message: “calibration”

File: install/sad_pkg/share/sad_pkg/urdf/description/test.xacro (robot description, xacro)
@@ -197,5 +197,5 @@
         <child link="link3"/>
         <origin xyz="0 0.205 0" rpy="0 3.14 3.14"/>
-        <axis xyz="0 1 0" />
+        <axis xyz="0 -1 0" />
         <limit effort="1000.0" velocity="10" lower="-3.14" upper="3.14" />
         <dynamics damping="100" friction="50" />
@@ -213,5 +213,5 @@
         <child link="link5"/>
         <origin xyz="0 0.0005 -0.202" rpy="1.57 0 1.57"/>
-        <axis xyz="0 1 0" />
+        <axis xyz="0 -1 0" />
         <limit effort="1000.0" velocity="10" lower="-3.14" upper="3.14" />
         <dynamics damping="100" friction="50" />

Commit message: “simulation_last”

File: install/sad_pkg/share/sad_pkg/urdf/description/test.xacro (robot description, xacro)
@@ -190,5 +190,5 @@
         <origin xyz="-0.004 0.018 0" rpy="0 0 0"/>
         <axis xyz="0 0 -1" />
-        <limit effort="1000.0" velocity="10" lower="-3.14" upper="3.14" />
+        <limit effort="1000.0" velocity="10" lower="-1.571" upper="1.571" />
         <dynamics damping="100" friction="50" />
     </joint>
@@ -206,5 +206,5 @@
         <origin xyz="0 -0.068 0.0015" rpy="-1.57 0 0"/>
         <axis xyz="0 -1 0" />
-        <limit effort="1000.0" velocity="10" lower="-3.14" upper="3.14" />
+        <limit effort="1000.0" velocity="10" lower="-2.094" upper="2.094" />
         <dynamics damping="100" friction="50" />
     </joint>
@@ -222,5 +222,5 @@
         <origin xyz="0 -0.053 0" rpy="1.57 1.57 0"/>
         <axis xyz="0 -1 0" />
-        <limit effort="1000.0" velocity="10" lower="-3.14" upper="3.14" />
+        <limit effort="1000.0" velocity="10" lower="-3.14" upper="0.524" />
         <dynamics damping="100" friction="50" />
     </joint>

Commit message: “dynamixel”

File: install/sad_pkg/share/sad_pkg/urdf/description/test.xacro (robot description, xacro)
@@ -190,5 +190,5 @@
         <origin xyz="-0.004 0.018 0" rpy="0 0 0"/>
         <axis xyz="0 0 -1" />
-        <limit effort="1000.0" velocity="10" lower="-1.571" upper="1.571" />
+        <limit effort="1000.0" velocity="10" lower="-3.14" upper="3.14" />
         <dynamics damping="100" friction="50" />
     </joint>
@@ -206,5 +206,5 @@
         <origin xyz="0 -0.068 0.0015" rpy="-1.57 0 0"/>
         <axis xyz="0 -1 0" />
-        <limit effort="1000.0" velocity="10" lower="-2.094" upper="2.094" />
+        <limit effort="1000.0" velocity="10" lower="-3.14" upper="3.14" />
         <dynamics damping="100" friction="50" />
     </joint>
@@ -222,5 +222,5 @@
         <origin xyz="0 -0.053 0" rpy="1.57 1.57 0"/>
         <axis xyz="0 -1 0" />
-        <limit effort="1000.0" velocity="10" lower="-3.14" upper="0.524" />
+        <limit effort="1000.0" velocity="10" lower="-3.14" upper="3.14" />
         <dynamics damping="100" friction="50" />
     </joint>
